Commit message: testing mount ori +45deg

File: src/custom_workcell/i40_workcell/urdf/workcell_macro.xacro (robot description, xacro)
@@ -52,5 +52,5 @@
       <parent link="table"/>
       <child link="robot_mount"/>
-      <origin xyz="0.0 0.0 0.0" rpy="0 0 0" />
+      <origin xyz="0.0 0.0 0.0" rpy="0 0 0.785" />
     </joint>
     <link name="femto_mount">
