Commit message: ur20workcell mount tune

File: src/custom_workcell/ur20_workcell/urdf/workcell_macro.xacro (robot description, xacro)
@@ -57,10 +57,10 @@
       <visual>
         <geometry>
-          <mesh filename="package://ur20_workcell/meshes/femto_mount.dae"/>
+          <mesh filename="package://ur20_workcell/meshes/ur20_bolt_mount_v2.dae"/>
         </geometry>
       </visual>
       <collision>
         <geometry>
-         <mesh filename="package://ur20_workcell/meshes/femto_mount.dae"/>
+         <mesh filename="package://ur20_workcell/meshes/ur20_bolt_mount_v2.dae"/>
         </geometry>
       </collision>

Commit message: UR20 macro update

File: src/custom_workcell/ur20_workcell/urdf/workcell_macro.xacro (robot description, xacro)
@@ -15,42 +15,59 @@
       <xacro:insert_block name="origin" />
       <parent link="${parent}" />
-      <child link="table" />
+      <child link="robot_base" />
     </joint>
-    <link name="table">
+    <link name="robot_base">
       <visual>
         <geometry>
-          <mesh filename="package://ur20_workcell/meshes/table.dae"/>
+          <mesh filename="package://ur20_workcell/meshes/robot_base.dae"/>
         </geometry>
-        <origin rpy="0 0 0" xyz="-0.125 0.475 -0.74"/>
+        <origin rpy="0 0 0" xyz="0.0 0.0 0.0"/>
       </visual>
       <collision>
         <geometry>
-          <mesh filename="package://ur20_workcell/meshes/table.dae"/>
+          <mesh filename="package://ur20_workcell/meshes/robot_base.dae"/>
         </geometry>
-        <origin rpy="0 0 0" xyz="-0.125 0.475 -0.74"/>
+        <origin rpy="0 0 0" xyz="0.0 0.0 0.0"/>
       </collision>
     </link>
-    <link name="wall">
+    <link name="handrail">
       <visual>
         <geometry>
-          <mesh filename="package://ur20_workcell/meshes/wall.dae"/>
+          <mesh filename="package://ur20_workcell/meshes/handrail.dae"/>
         </geometry>
       </visual>
       <collision>
         <geometry>
-         <mesh filename="package://ur20_workcell/meshes/wall.dae"/>
+         <mesh filename="package://ur20_workcell/meshes/handrail.dae"/>
         </geometry>
       </collision>
     </link>
-    <joint name="base_to_wall" type="fixed">
-      <parent link="table"/>
-      <child link="wall"/>
-      <origin xyz="0 -0.67 -0.74"/>
+    <joint name="base_to_handrail" type="fixed">
+      <parent link="robot_base"/>
+      <child link="handrail"/>
+      <origin xyz="0 0 0"/>
     </joint>
-    <link name="robot_mount"/>
-    <joint name="base_to_robot_mount" type="fixed">
-      <parent link="table"/>
-      <child link="robot_mount"/>
-      <origin xyz="0.0 0.0 0.0" rpy="0 0 0.785" />
+    <link name="control_box">
+      <visual>
+        <geometry>
+          <mesh filename="package://ur20_workcell/meshes/control_box.dae"/>
+        </geometry>
+      </visual>
+      <collision>
+        <geometry>
+         <mesh filename="package://ur20_workcell/meshes/control_box.dae"/>
+        </geometry>
+      </collision>
+    </link>
+    <joint name="base_to_control_box" type="fixed">
+      <parent link="robot_base"/>
+      <child link="control_box"/>
+      <origin xyz="0 0 0"/>
+    </joint>
+    <link name="table"/>
+    <joint name="base_to_table" type="fixed">
+      <parent link="robot_base"/>
+      <child link="table"/>
+      <origin xyz="0.0 0.6 0.0" rpy="0 0 0" />
     </joint>
     <link name="femto_mount">

Commit message: macro_update_UR20workcell

File: src/custom_workcell/ur20_workcell/urdf/workcell_macro.xacro (robot description, xacro)
@@ -31,4 +31,10 @@
       </collision>
     </link>
+    <link name="robot_mount"/>
+    <joint name="base_to_robot_mount" type="fixed">
+      <parent link="robot_base"/>
+      <child link="robot_mount"/>
+      <origin xyz="0.0 0.0 0.0" rpy="0 0 0.0" />
+    </joint>
     <link name="handrail">
       <visual>
@@ -65,5 +71,16 @@
       <origin xyz="0 0 0"/>
     </joint>
-    <link name="table"/>
+    <link name="table">
+      <visual>
+        <geometry>
+          <mesh filename="package://ur20_workcell/meshes/table.dae"/>
+        </geometry>
+      </visual>
+      <collision>
+        <geometry>
+         <mesh filename="package://ur20_workcell/meshes/table.dae"/>
+        </geometry>
+      </collision>
+    </link>
     <joint name="base_to_table" type="fixed">
       <parent link="robot_base"/>

Commit message: UR20 real hardware working in kinematic demo cpp

File: src/custom_workcell/ur20_workcell/urdf/workcell_macro.xacro (robot description, xacro)
@@ -35,5 +35,5 @@
       <parent link="robot_base"/>
       <child link="robot_mount"/>
-      <origin xyz="0.0 0.0 0.0" rpy="0 0 0.0" />
+      <origin xyz="0.0 0.0 0.0" rpy="0 0 3.1415" />
     </joint>
     <link name="handrail">

Commit message: URDF updated

File: src/custom_workcell/ur20_workcell/urdf/workcell_macro.xacro (robot description, xacro)
@@ -103,5 +103,5 @@
       <parent link="${ur_type}_tool0"/>
       <child link="femto_mount"/>
-      <origin xyz="0 0 0"/>
+      <origin xyz="0 0 0" rpy="0 0 -0.5235"/>
     </joint>
     <!--This will create the specific robot-->
@@ -122,5 +122,5 @@
       use_nominal_extrinsics="true"
     >
-      <origin xyz="0 0.0555 0.0103" rpy="0 0 1.5708" />
+      <origin xyz="0.027 0.048 0.0103" rpy="0 0 1.0472" />
     </xacro:femto_bolt>
   </xacro:macro>

Commit message: Urdf Update

File: src/custom_workcell/ur20_workcell/urdf/workcell_macro.xacro (robot description, xacro)
@@ -69,5 +69,5 @@
       <parent link="robot_base"/>
       <child link="control_box"/>
-      <origin xyz="0 0 0"/>
+      <origin xyz="0 0 0.0"/>
     </joint>
     <link name="table">
@@ -86,5 +86,28 @@
       <parent link="robot_base"/>
       <child link="table"/>
-      <origin xyz="0.0 0.6 0.0" rpy="0 0 0" />
+      <origin xyz="-0.15 0.5 -0.08" rpy="0 0 0" />
+    </joint>
+    <!-- Desktop (table) -->
+    <link name="desktop">
+      <visual>
+        <origin xyz="0 0 0"/>
+        <geometry>
+          <box size="2.0 1.2 0.90"/>
+        </geometry>
+        <material name="DesktopGrey">
+          <color rgba="0.6 0.6 0.6 1.0"/>
+        </material>
+      </visual>
+      <collision>
+        <origin xyz="0 0 0"/>
+        <geometry>
+          <box size="2.0 1.2 0.90"/>
+        </geometry>
+      </collision>
+    </link>
+    <joint name="base_to_desktop" type="fixed">
+      <parent link="robot_base"/>
+      <child link="desktop"/>
+      <origin xyz="1.7 0 -0.48" rpy="0 0 0"/>
     </joint>
     <link name="femto_mount">

Commit message: handeye integration to previous convention

File: src/custom_workcell/ur20_workcell/urdf/workcell_macro.xacro (robot description, xacro)
@@ -105,4 +105,14 @@
       <origin xyz="0 0 0" rpy="0 0 -0.5235"/>
     </joint>
+    <!-- Fixed frame for calibrated camera pose relative to tool0 -->
+    <link name="femto_color_optical_calib"/>
+    <joint name="tool0_to_femto_color_optical_calib" type="fixed">
+      <parent link="${ur_type}_tool0"/>
+      <child link="femto_color_optical_calib"/>
+      <!-- Origin is tool0 -> camera (meters, radians).
+          RPY is extrinsic X-Y-Z (roll, pitch, yaw) as in URDF. -->
+      <origin xyz="0.0675963 0.0564383 0.0319683"
+              rpy="-1.5641113421 -0.0089024576 -0.5209877605"/>
+    </joint>
     <!--This will create the specific robot-->
     <xacro:ur_robot

Commit message: update extruder_tcp eef on urdf

File: src/custom_workcell/ur20_workcell/urdf/workcell_macro.xacro (robot description, xacro)
@@ -86,5 +86,5 @@
       <parent link="robot_base"/>
       <child link="table"/>
-      <origin xyz="0.0 0.6 0.0" rpy="0 0 0" />
+      <origin xyz="-0.15 0.5 -0.08" rpy="0 0 0" />
     </joint>
     <link name="femto_mount">
@@ -115,4 +115,14 @@
               rpy="-1.5641113421 -0.0089024576 -0.5209877605"/>
     </joint>
+    <!-- Fixed frame for calibrated Extruder tcp pose relative to tool0 -->
+    <link name="extruder_tcp"/>
+    <joint name="tool0_to_extruder_tcp" type="fixed">
+      <parent link="${ur_type}_tool0"/>
+      <child link="extruder_tcp"/>
+      <!-- Origin is tool0 -> camera (meters, radians).
+          RPY is extrinsic X-Y-Z (roll, pitch, yaw) as in URDF. -->
+      <origin xyz="0.0094 0.2272 0.07784"
+              rpy="1.5641113421 0.0 0.0"/>
+    </joint>
     <!--This will create the specific robot-->
     <xacro:ur_robot

Commit message: Print and move via commands class

File: src/custom_workcell/ur20_workcell/urdf/workcell_macro.xacro (robot description, xacro)
@@ -35,5 +35,5 @@
       <parent link="robot_base"/>
       <child link="robot_mount"/>
-      <origin xyz="0.0 0.0 0.0" rpy="0 0 3.1415" />
+      <origin xyz="0.0 0.0 0.0" rpy="0 0 3.1415926" />
     </joint>
     <link name="handrail">
@@ -120,5 +120,5 @@
       <parent link="${ur_type}_tool0"/>
       <child link="extruder_tcp"/>
-      <!-- Origin is tool0 -> camera (meters, radians).
+      <!-- Origin is tool0 -> extruder(meters, radians).
           RPY is extrinsic X-Y-Z (roll, pitch, yaw) as in URDF. -->
       <origin xyz="0.0094 0.2272 0.07784"

Commit message: 3 dots print demo

File: src/custom_workcell/ur20_workcell/urdf/workcell_macro.xacro (robot description, xacro)
@@ -122,5 +122,5 @@
       <!-- Origin is tool0 -> extruder(meters, radians).
           RPY is extrinsic X-Y-Z (roll, pitch, yaw) as in URDF. -->
-      <origin xyz="0.0094 0.2272 0.07784"
+      <origin xyz="0.00094 0.2272 0.07784"
               rpy="1.5641113421 0.0 0.0"/>
     </joint>

Commit message: clay extruder in workcell model

File: src/custom_workcell/ur20_workcell/urdf/workcell_macro.xacro (robot description, xacro)
@@ -88,13 +88,13 @@
       <origin xyz="-0.15 0.5 -0.08" rpy="0 0 0" />
     </joint>
-    <link name="femto_mount">
+    <link name="clay_extruder">
       <visual>
         <geometry>
-          <mesh filename="package://ur20_workcell/meshes/ur20_bolt_mount_v2.dae"/>
+          <mesh filename="package://ur20_workcell/meshes/clay_extruder.dae"/>
         </geometry>
       </visual>
       <collision>
         <geometry>
-         <mesh filename="package://ur20_workcell/meshes/ur20_bolt_mount_v2.dae"/>
+         <mesh filename="package://ur20_workcell/meshes/clay_extruder.dae"/>
         </geometry>
       </collision>
@@ -102,6 +102,6 @@
     <joint name="base_to_tool0" type="fixed">
       <parent link="${ur_type}_tool0"/>
-      <child link="femto_mount"/>
-      <origin xyz="0 0 0" rpy="0 0 -0.5235"/>
+      <child link="clay_extruder"/>
+      <origin xyz="0 0 0" rpy="0 0 0"/>
     </joint>
     <!-- Fixed frame for calibrated camera pose relative to tool0 -->

Commit message: workcell adjustment

File: src/custom_workcell/ur20_workcell/urdf/workcell_macro.xacro (robot description, xacro)
@@ -91,10 +91,10 @@
       <visual>
         <geometry>
-          <mesh filename="package://ur20_workcell/meshes/clay_extruder.dae"/>
+          <mesh filename="package://ur20_workcell/meshes/clay_extruder_cam.dae"/>
         </geometry>
       </visual>
       <collision>
         <geometry>
-         <mesh filename="package://ur20_workcell/meshes/clay_extruder.dae"/>
+         <mesh filename="package://ur20_workcell/meshes/clay_extruder_cam.dae"/>
         </geometry>
       </collision>
@@ -142,5 +142,5 @@
       use_nominal_extrinsics="true"
     >
-      <origin xyz="0.027 0.048 0.0103" rpy="0 0 1.0472" />
+      <origin xyz="0.0 0.178 -0.051" rpy="0 3.141592 0" />
     </xacro:femto_bolt>
   </xacro:macro>

Commit message: urdf update

File: src/custom_workcell/ur20_workcell/urdf/workcell_macro.xacro (robot description, xacro)
@@ -142,5 +142,5 @@
       use_nominal_extrinsics="true"
     >
-      <origin xyz="0.0 0.178 -0.051" rpy="0 3.141592 0" />
+      <origin xyz="0.0 0.164 -0.051" rpy="0 3.141592 0" />
     </xacro:femto_bolt>
   </xacro:macro>

Commit message: Urdf updates

File: src/custom_workcell/ur20_workcell/urdf/workcell_macro.xacro (robot description, xacro)
@@ -112,6 +112,6 @@
       <!-- Origin is tool0 -> camera (meters, radians).
           RPY is extrinsic X-Y-Z (roll, pitch, yaw) as in URDF. -->
-      <origin xyz="0.0675963 0.0564383 0.0319683"
-              rpy="-1.5641113421 -0.0089024576 -0.5209877605"/>
+      <origin xyz="-0.0445562   0.17385712 -0.07569992"
+               quat="0.01124485 0.7136558  0.70033581 0.00993505"/>
     </joint>
     <!-- Fixed frame for calibrated Extruder tcp pose relative to tool0 -->
@@ -142,5 +142,5 @@
       use_nominal_extrinsics="true"
     >
-      <origin xyz="0.0 0.164 -0.051" rpy="0 3.141592 0" />
+      <origin xyz="0.0 0.164 -0.051" rpy="0 3.141592 -1.5707964" />
     </xacro:femto_bolt>
   </xacro:macro>

Commit message: urdf new ir calib frame and handeye scripts

File: src/custom_workcell/ur20_workcell/urdf/workcell_macro.xacro (robot description, xacro)
@@ -112,6 +112,16 @@
       <!-- Origin is tool0 -> camera (meters, radians).
           RPY is extrinsic X-Y-Z (roll, pitch, yaw) as in URDF. -->
-      <origin xyz="-0.0445562   0.17385712 -0.07569992"
-               rpy="1.589 -0.00152 3.111"/>
+      <origin xyz="-0.00833796  0.17520484 -0.07128864"
+               rpy="1.603 0.006 -3.097"/>
+    </joint>
+    <!-- Fixed frame for calibrated camera pose relative to tool0 -->
+    <link name="femto_ir_optical_calib"/>
+    <joint name="tool0_to_femto_ir_optical_calib" type="fixed">
+      <parent link="${ur_type}_tool0"/>
+      <child link="femto_ir_optical_calib"/>
+      <!-- Origin is tool0 -> camera (meters, radians).
+          RPY is extrinsic X-Y-Z (roll, pitch, yaw) as in URDF. -->
+      <origin xyz="0.02985754  0.1759846  -0.07227334"
+               rpy="1.499 0.001 -3.082"/>
     </joint>
     <!-- Fixed frame for calibrated Extruder tcp pose relative to tool0 -->

Commit message: Handeye calibration scripts adjusted

File: src/custom_workcell/ur20_workcell/urdf/workcell_macro.xacro (robot description, xacro)
@@ -112,6 +112,6 @@
       <!-- Origin is tool0 -> camera (meters, radians).
           RPY is extrinsic X-Y-Z (roll, pitch, yaw) as in URDF. -->
-      <origin xyz="-0.00833796  0.17520484 -0.07128864"
-               rpy="1.603 0.006 -3.097"/>
+      <origin xyz="-0.03158908  0.1747814  -0.07149736"
+               rpy="1.599 0.002 -3.139"/>
     </joint>
     <!-- Fixed frame for calibrated camera pose relative to tool0 -->
@@ -122,6 +122,6 @@
       <!-- Origin is tool0 -> camera (meters, radians).
           RPY is extrinsic X-Y-Z (roll, pitch, yaw) as in URDF. -->
-      <origin xyz="0.02985754  0.1759846  -0.07227334"
-               rpy="1.499 0.001 -3.082"/>
+      <origin xyz="0.00028979  0.17421966 -0.07240817"
+               rpy="1.496 -0.005 -3.140"/>
     </joint>
     <!-- Fixed frame for calibrated Extruder tcp pose relative to tool0 -->

Commit message: urdf update with eef_v2

File: src/custom_workcell/ur20_workcell/urdf/workcell_macro.xacro (robot description, xacro)
@@ -91,10 +91,10 @@
       <visual>
         <geometry>
-          <mesh filename="package://ur20_workcell/meshes/clay_extruder_cam.dae"/>
+          <mesh filename="package://ur20_workcell/meshes/clay_extruder_cam_v2.dae"/>
         </geometry>
       </visual>
       <collision>
         <geometry>
-         <mesh filename="package://ur20_workcell/meshes/clay_extruder_cam.dae"/>
+         <mesh filename="package://ur20_workcell/meshes/clay_extruder_cam_v2.dae"/>
         </geometry>
       </collision>
@@ -152,5 +152,5 @@
       use_nominal_extrinsics="true"
     >
-      <origin xyz="0.0 0.164 -0.051" rpy="0 3.141592 -1.5707964" />
+      <origin xyz="0.0 0.128 -0.014" rpy="0 3.141592 -1.5707964" />
     </xacro:femto_bolt>
   </xacro:macro>

Commit message: handeye update to new framework loose urdf update

File: src/custom_workcell/ur20_workcell/urdf/workcell_macro.xacro (robot description, xacro)
@@ -112,6 +112,6 @@
       <!-- Origin is tool0 -> camera (meters, radians).
           RPY is extrinsic X-Y-Z (roll, pitch, yaw) as in URDF. -->
-      <origin xyz="-0.03158908  0.1747814  -0.07149736"
-               rpy="1.599 0.002 -3.139"/>
+      <origin xyz="-0.03056191  0.15579223 -0.0323924"
+               rpy="1.5842179087 0.0069115038 -3.1414530273"/>
     </joint>
     <!-- Fixed frame for calibrated camera pose relative to tool0 -->
@@ -122,6 +122,6 @@
       <!-- Origin is tool0 -> camera (meters, radians).
           RPY is extrinsic X-Y-Z (roll, pitch, yaw) as in URDF. -->
-      <origin xyz="0.00028979  0.17421966 -0.07240817"
-               rpy="1.496 -0.005 -3.140"/>
+      <origin xyz="0.00406406  0.14887232 -0.03403896"
+               rpy="1.4770372394 -0.0096691241 -3.1290437363"/>
     </joint>
     <!-- Fixed frame for calibrated Extruder tcp pose relative to tool0 -->

Commit message: urdf update tcp and reconstruction intrinsics / folder link

File: src/custom_workcell/ur20_workcell/urdf/workcell_macro.xacro (robot description, xacro)
@@ -112,6 +112,6 @@
       <!-- Origin is tool0 -> camera (meters, radians).
           RPY is extrinsic X-Y-Z (roll, pitch, yaw) as in URDF. -->
-      <origin xyz="-0.03056191  0.15579223 -0.0323924"
-               rpy="1.5842179087 0.0069115038 -3.1414530273"/>
+      <origin xyz="-0.02920643  0.15712499 -0.03328242"
+               rpy="1.5843051752 0.0075921822 -3.1405280027"/>
     </joint>
     <!-- Fixed frame for calibrated camera pose relative to tool0 -->
@@ -122,6 +122,6 @@
       <!-- Origin is tool0 -> camera (meters, radians).
           RPY is extrinsic X-Y-Z (roll, pitch, yaw) as in URDF. -->
-      <origin xyz="0.00406406  0.14887232 -0.03403896"
-               rpy="1.4770372394 -0.0096691241 -3.1290437363"/>
+      <origin xyz="0.00589702  0.16138198 -0.04035296"
+               rpy="1.4738781934 0.0028099801 -3.1294800686"/>
     </joint>
     <!-- Fixed frame for calibrated Extruder tcp pose relative to tool0 -->
@@ -132,5 +132,5 @@
       <!-- Origin is tool0 -> extruder(meters, radians).
           RPY is extrinsic X-Y-Z (roll, pitch, yaw) as in URDF. -->
-      <origin xyz="0.00094 0.2272 0.07784"
+      <origin xyz="-0.00094 0.24496 0.06159"
               rpy="1.5641113421 0.0 0.0"/>
     </joint>

Commit message: handeye improvements

File: src/custom_workcell/ur20_workcell/urdf/workcell_macro.xacro (robot description, xacro)
@@ -112,6 +112,6 @@
       <!-- Origin is tool0 -> camera (meters, radians).
           RPY is extrinsic X-Y-Z (roll, pitch, yaw) as in URDF. -->
-      <origin xyz="-0.02920643  0.15712499 -0.03328242"
-               rpy="1.5843051752 0.0075921822 -3.1405280027"/>
+      <origin xyz="-0.03041263  0.15675367 -0.03452134"
+               rpy="1.5836070435 0.0075223691 -3.1412784943"/>
     </joint>
     <!-- Fixed frame for calibrated camera pose relative to tool0 -->
@@ -122,6 +122,6 @@
       <!-- Origin is tool0 -> camera (meters, radians).
           RPY is extrinsic X-Y-Z (roll, pitch, yaw) as in URDF. -->
-      <origin xyz="0.00589702  0.16138198 -0.04035296"
-               rpy="1.4738781934 0.0028099801 -3.1294800686"/>
+      <origin xyz="0.00180271  0.15873923 -0.03501765"
+               rpy=" 1.4796203267 0.0010471976 -3.1372642370 "/>
     </joint>
     <!-- Fixed frame for calibrated Extruder tcp pose relative to tool0 -->

Commit message: handeye formatting

File: src/custom_workcell/ur20_workcell/urdf/workcell_macro.xacro (robot description, xacro)
@@ -113,5 +113,5 @@
           RPY is extrinsic X-Y-Z (roll, pitch, yaw) as in URDF. -->
       <origin xyz="-0.03041263  0.15675367 -0.03452134"
-               rpy="1.5836070435 0.0075223691 -3.1412784943"/>
+               rpy="1.583606 0.007528 -3.141280"/>
     </joint>
     <!-- Fixed frame for calibrated camera pose relative to tool0 -->
@@ -122,6 +122,6 @@
       <!-- Origin is tool0 -> camera (meters, radians).
           RPY is extrinsic X-Y-Z (roll, pitch, yaw) as in URDF. -->
-      <origin xyz="0.00180271  0.15873923 -0.03501765"
-               rpy=" 1.4796203267 0.0010471976 -3.1372642370 "/>
+      <origin xyz="0.00203272  0.15910973 -0.03529811"
+               rpy=" 1.479059 0.001322 -3.137201 "/>
     </joint>
     <!-- Fixed frame for calibrated Extruder tcp pose relative to tool0 -->

Commit message: urdf and print updates

File: src/custom_workcell/ur20_workcell/urdf/workcell_macro.xacro (robot description, xacro)
@@ -91,10 +91,10 @@
       <visual>
         <geometry>
-          <mesh filename="package://ur20_workcell/meshes/clay_extruder_cam_v2.dae"/>
+          <mesh filename="package://ur20_workcell/meshes/clay_extruder_cam_calibrated_v2.dae"/>
         </geometry>
       </visual>
       <collision>
         <geometry>
-         <mesh filename="package://ur20_workcell/meshes/clay_extruder_cam_v2.dae"/>
+         <mesh filename="package://ur20_workcell/meshes/clay_extruder_cam_calibrated_v2.dae"/>
         </geometry>
       </collision>
@@ -132,5 +132,5 @@
       <!-- Origin is tool0 -> extruder(meters, radians).
           RPY is extrinsic X-Y-Z (roll, pitch, yaw) as in URDF. -->
-      <origin xyz="-0.00094 0.24496 0.06159"
+      <origin xyz="-0.00233 0.25763 0.06222"
               rpy="1.5641113421 0.0 0.0"/>
     </joint>

Commit message: handeye script update

File: src/custom_workcell/ur20_workcell/urdf/workcell_macro.xacro (robot description, xacro)
@@ -112,6 +112,6 @@
       <!-- Origin is tool0 -> camera (meters, radians).
           RPY is extrinsic X-Y-Z (roll, pitch, yaw) as in URDF. -->
-      <origin xyz="-0.03041263  0.15675367 -0.03452134"
-               rpy="1.583606 0.007528 -3.141280"/>
+      <origin xyz="-0.0308383   0.15721051 -0.03262603"
+               rpy="1.5843028 0.0077415 -3.1384045"/>
     </joint>
     <!-- Fixed frame for calibrated camera pose relative to tool0 -->
@@ -122,6 +122,6 @@
       <!-- Origin is tool0 -> camera (meters, radians).
           RPY is extrinsic X-Y-Z (roll, pitch, yaw) as in URDF. -->
-      <origin xyz="0.00203272  0.15910973 -0.03529811"
-               rpy=" 1.479059 0.001322 -3.137201 "/>
+      <origin xyz="0.00199305  0.16085472 -0.03313815"
+               rpy=" 1.4803456 0.0033778 -3.1342829"/>
     </joint>
     <!-- Fixed frame for calibrated Extruder tcp pose relative to tool0 -->
