Commit message: Code cleanup + utility session + Print node updates

File: src/custom_workcell/ur20_workcell/urdf/workcell_macro.xacro (robot description, xacro)
@@ -112,6 +112,6 @@
       <!-- Origin is tool0 -> camera (meters, radians).
           RPY is extrinsic X-Y-Z (roll, pitch, yaw) as in URDF. -->
-      <origin xyz="-0.0308383   0.15721051 -0.03262603"
-               rpy="1.5843028 0.0077415 -3.1384045"/>
+      <origin xyz="-0.03107523  0.15939788 -0.03590129"
+               rpy="1.5841069 0.0083596 -3.1385739"/>
     </joint>
     <!-- Fixed frame for calibrated camera pose relative to tool0 -->
@@ -122,6 +122,6 @@
       <!-- Origin is tool0 -> camera (meters, radians).
           RPY is extrinsic X-Y-Z (roll, pitch, yaw) as in URDF. -->
-      <origin xyz="0.00199305  0.16085472 -0.03313815"
-               rpy=" 1.4803456 0.0033778 -3.1342829"/>
+      <origin xyz="0.0004368   0.16222267 -0.03703682"
+               rpy=" 1.4800043 0.0037694 -3.1355591"/>
     </joint>
     <!-- Fixed frame for calibrated Extruder tcp pose relative to tool0 -->

Commit message: handeye validation and urdf camera extrinsics update

File: src/custom_workcell/ur20_workcell/urdf/workcell_macro.xacro (robot description, xacro)
@@ -112,6 +112,6 @@
       <!-- Origin is tool0 -> camera (meters, radians).
           RPY is extrinsic X-Y-Z (roll, pitch, yaw) as in URDF. -->
-      <origin xyz="-0.03107523  0.15939788 -0.03590129"
-               rpy="1.5841069 0.0083596 -3.1385739"/>
+      <origin xyz="-0.031924016245898724 0.15743490860827325 -0.03357736917378262"
+               rpy="1.5839457680003415 0.00827678727740544 -3.138847872677128"/>
     </joint>
     <!-- Fixed frame for calibrated camera pose relative to tool0 -->
@@ -122,6 +122,6 @@
       <!-- Origin is tool0 -> camera (meters, radians).
           RPY is extrinsic X-Y-Z (roll, pitch, yaw) as in URDF. -->
-      <origin xyz="0.0004368   0.16222267 -0.03703682"
-               rpy=" 1.4800043 0.0037694 -3.1355591"/>
+      <origin xyz="0.0003127735651572818 0.1612232972598608 -0.03475076070075697"
+               rpy=" 1.4795689717799185 0.0028874147759252455 -3.135140027256738"/>
     </joint>
     <!-- Fixed frame for calibrated Extruder tcp pose relative to tool0 -->

Commit message: URDF WORKCELL UPDATE FOR MEGA

File: src/custom_workcell/ur20_workcell/urdf/workcell_macro.xacro (robot description, xacro)
@@ -91,10 +91,10 @@
       <visual>
         <geometry>
-          <mesh filename="package://ur20_workcell/meshes/clay_extruder_cam_calibrated_v2.dae"/>
+          <mesh filename="package://ur20_workcell/meshes/clay_extruder_cam_calibrated_v4.dae"/>
         </geometry>
       </visual>
       <collision>
         <geometry>
-         <mesh filename="package://ur20_workcell/meshes/clay_extruder_cam_calibrated_v2.dae"/>
+         <mesh filename="package://ur20_workcell/meshes/clay_extruder_cam_calibrated_v4.dae"/>
         </geometry>
       </collision>
@@ -112,6 +112,6 @@
       <!-- Origin is tool0 -> camera (meters, radians).
           RPY is extrinsic X-Y-Z (roll, pitch, yaw) as in URDF. -->
-      <origin xyz="-0.031924016245898724 0.15743490860827325 -0.03357736917378262"
-               rpy="1.5839457680003415 0.00827678727740544 -3.138847872677128"/>
+      <origin xyz="-0.05996046861797611 0.1776607683506138 0.09264273877852516"
+               rpy="0.6799468880371341 -1.5573071040676396 -2.241519026643666"/>
     </joint>
     <!-- Fixed frame for calibrated camera pose relative to tool0 -->
@@ -122,6 +122,6 @@
       <!-- Origin is tool0 -> camera (meters, radians).
           RPY is extrinsic X-Y-Z (roll, pitch, yaw) as in URDF. -->
-      <origin xyz="0.0003127735651572818 0.1612232972598608 -0.03475076070075697"
-               rpy=" 1.4795689717799185 0.0028874147759252455 -3.135140027256738"/>
+      <origin xyz="-0.06064789409656456 0.180481984883551 0.06164066350253106"
+               rpy="0.4304040763127037 -1.5584296812405685 -2.09948979178602"/>
     </joint>
     <!-- Fixed frame for calibrated Extruder tcp pose relative to tool0 -->
@@ -132,5 +132,5 @@
       <!-- Origin is tool0 -> extruder(meters, radians).
           RPY is extrinsic X-Y-Z (roll, pitch, yaw) as in URDF. -->
-      <origin xyz="-0.00233 0.25763 0.06222"
+      <origin xyz="0.0469 0.28199 0.06276"
               rpy="1.5641113421 0.0 0.0"/>
     </joint>
@@ -152,5 +152,5 @@
       use_nominal_extrinsics="true"
     >
-      <origin xyz="0.0 0.128 -0.014" rpy="0 3.141592 -1.5707964" />
+      <origin xyz="-0.03816 0.1486 0.062017" rpy="-1.5707964 0 1.5707964" />
     </xacro:femto_bolt>
   </xacro:macro>

Commit message: new hand eye and some stuff in my scripts in tsdf

File: src/custom_workcell/ur20_workcell/urdf/workcell_macro.xacro (robot description, xacro)
@@ -112,6 +112,6 @@
       <!-- Origin is tool0 -> camera (meters, radians).
           RPY is extrinsic X-Y-Z (roll, pitch, yaw) as in URDF. -->
-      <origin xyz="-0.05996046861797611 0.1776607683506138 0.09264273877852516"
-               rpy="0.6799468880371341 -1.5573071040676396 -2.241519026643666"/>
+      <origin xyz="-0.0596693318086239 0.17834453583169566 0.09396434130245321"
+               rpy="0.6120233973067307 -1.5597566066936388 -2.1737006287734144"/>
     </joint>
     <!-- Fixed frame for calibrated camera pose relative to tool0 -->
@@ -122,6 +122,6 @@
       <!-- Origin is tool0 -> camera (meters, radians).
           RPY is extrinsic X-Y-Z (roll, pitch, yaw) as in URDF. -->
-      <origin xyz="-0.06064789409656456 0.180481984883551 0.06164066350253106"
-               rpy="0.4304040763127037 -1.5584296812405685 -2.09948979178602"/>
+      <origin xyz="-0.06091216464344758 0.18117284946693304 0.05983544324216165"
+               rpy="0.18011085182694897 -1.5576080190564232 -1.84996888512795"/>
     </joint>
     <!-- Fixed frame for calibrated Extruder tcp pose relative to tool0 -->

Commit message: tcp and handeye calibration

File: src/custom_workcell/ur20_workcell/urdf/workcell_macro.xacro (robot description, xacro)
@@ -112,6 +112,6 @@
       <!-- Origin is tool0 -> camera (meters, radians).
           RPY is extrinsic X-Y-Z (roll, pitch, yaw) as in URDF. -->
-      <origin xyz="-0.0596693318086239 0.17834453583169566 0.09396434130245321"
-               rpy="0.6120233973067307 -1.5597566066936388 -2.1737006287734144"/>
+      <origin xyz="-0.059067526871075304 0.17829638444677057 0.09322089637670121"
+               rpy="0.5929766178458789 -1.5588222818238573 -2.1542935523812377"/>
     </joint>
     <!-- Fixed frame for calibrated camera pose relative to tool0 -->
@@ -122,6 +122,6 @@
       <!-- Origin is tool0 -> camera (meters, radians).
           RPY is extrinsic X-Y-Z (roll, pitch, yaw) as in URDF. -->
-      <origin xyz="-0.06091216464344758 0.18117284946693304 0.05983544324216165"
-               rpy="0.18011085182694897 -1.5576080190564232 -1.84996888512795"/>
+      <origin xyz="-0.06003225386528856 0.18114945673097352 0.06087181278791609"
+               rpy="0.23839553386181933 -1.558848276604893 -1.907707163639687"/>
     </joint>
     <!-- Fixed frame for calibrated Extruder tcp pose relative to tool0 -->
@@ -132,5 +132,5 @@
       <!-- Origin is tool0 -> extruder(meters, radians).
           RPY is extrinsic X-Y-Z (roll, pitch, yaw) as in URDF. -->
-      <origin xyz="0.0469 0.28199 0.06276"
+      <origin xyz="0.04733 0.28151 0.06228"
               rpy="1.5641113421 0.0 0.0"/>
     </joint>

Commit message: updated Handeye

File: src/custom_workcell/ur20_workcell/urdf/workcell_macro.xacro (robot description, xacro)
@@ -112,5 +112,5 @@
       <!-- Origin is tool0 -> camera (meters, radians).
           RPY is extrinsic X-Y-Z (roll, pitch, yaw) as in URDF. -->
-      <origin xyz="-0.059067526871075304 0.17829638444677057 0.09322089637670121"
+      <origin xyz="-0.059070068624449495 0.17914822584247272 0.09389743100591508"
                rpy="0.5929766178458789 -1.5588222818238573 -2.1542935523812377"/>
     </joint>
@@ -122,6 +122,6 @@
       <!-- Origin is tool0 -> camera (meters, radians).
           RPY is extrinsic X-Y-Z (roll, pitch, yaw) as in URDF. -->
-      <origin xyz="-0.06003225386528856 0.18114945673097352 0.06087181278791609"
-               rpy="0.23839553386181933 -1.558848276604893 -1.907707163639687"/>
+      <origin xyz="-0.06063506182578694 0.18168392383222384 0.0611143068526563"
+               rpy="0.10416277338198654 -1.5588723769304802 -1.7749299646347731"/>
     </joint>
     <!-- Fixed frame for calibrated Extruder tcp pose relative to tool0 -->

Commit message: workcell ram urdf update, handeye v5 py

File: src/custom_workcell/ur20_workcell/urdf/workcell_macro.xacro (robot description, xacro)
@@ -91,10 +91,10 @@
       <visual>
         <geometry>
-          <mesh filename="package://ur20_workcell/meshes/clay_extruder_cam_calibrated_v4.dae"/>
+          <mesh filename="package://ur20_workcell/meshes/ram_extruder_v2_simplified.dae"/>
         </geometry>
       </visual>
       <collision>
         <geometry>
-         <mesh filename="package://ur20_workcell/meshes/clay_extruder_cam_calibrated_v4.dae"/>
+         <mesh filename="package://ur20_workcell/meshes/ram_extruder_v2_simplified.dae"/>
         </geometry>
       </collision>
@@ -112,6 +112,6 @@
       <!-- Origin is tool0 -> camera (meters, radians).
           RPY is extrinsic X-Y-Z (roll, pitch, yaw) as in URDF. -->
-      <origin xyz="-0.059070068624449495 0.17914822584247272 0.09389743100591508"
-               rpy="0.5929766178458789 -1.5588222818238573 -2.1542935523812377"/>
+      <origin xyz="-0.03402996922467966 0.2970228148142489 -0.04855763948018441"
+               rpy="1.5799620345834504 -0.00404503983534954 -3.1063953966275766"/>
     </joint>
     <!-- Fixed frame for calibrated camera pose relative to tool0 -->
@@ -122,6 +122,6 @@
       <!-- Origin is tool0 -> camera (meters, radians).
           RPY is extrinsic X-Y-Z (roll, pitch, yaw) as in URDF. -->
-      <origin xyz="-0.06063506182578694 0.18168392383222384 0.0611143068526563"
-               rpy="0.10416277338198654 -1.5588723769304802 -1.7749299646347731"/>
+      <origin xyz="-0.004171269533157492 0.3005070159435434 -0.05050934664329281"
+               rpy="1.4706191997841613 -0.011294149359347028 -3.108643277714379"/>
     </joint>
     <!-- Fixed frame for calibrated Extruder tcp pose relative to tool0 -->
@@ -132,5 +132,5 @@
       <!-- Origin is tool0 -> extruder(meters, radians).
           RPY is extrinsic X-Y-Z (roll, pitch, yaw) as in URDF. -->
-      <origin xyz="0.04733 0.28151 0.06228"
+      <origin xyz="-0.00391 0.47471 0.08024"
               rpy="1.5641113421 0.0 0.0"/>
     </joint>
@@ -152,5 +152,5 @@
       use_nominal_extrinsics="true"
     >
-      <origin xyz="-0.03816 0.1486 0.062017" rpy="-1.5707964 0 1.5707964" />
+      <origin xyz="0 0.260 -0.03" rpy="3.14159 0 1.5707964" />
     </xacro:femto_bolt>
   </xacro:macro>

Commit message: primt yaml and scan orchestrator file

File: src/custom_workcell/ur20_workcell/urdf/workcell_macro.xacro (robot description, xacro)
@@ -86,5 +86,5 @@
       <parent link="robot_base"/>
       <child link="table"/>
-      <origin xyz="-0.15 0.5 -0.08" rpy="0 0 0" />
+      <origin xyz="-0.15 0.5 -1.08" rpy="0 0 0" />
     </joint>
     <link name="clay_extruder">
