Commit message: handeye and tcp calibrated

File: src/custom_workcell/ur20_workcell/urdf/workcell_macro.xacro (robot description, xacro)
@@ -112,6 +112,6 @@
       <!-- Origin is tool0 -> camera (meters, radians).
           RPY is extrinsic X-Y-Z (roll, pitch, yaw) as in URDF. -->
-      <origin xyz="-0.03402996922467966 0.2970228148142489 -0.04855763948018441"
-               rpy="1.5799620345834504 -0.00404503983534954 -3.1063953966275766"/>
+      <origin xyz="-0.034063681747165384 0.2956667467761771 -0.04632604563225764"
+               rpy="1.5797083152416658 -0.0024684364752196597 -3.109366333302816"/>
     </joint>
     <!-- Fixed frame for calibrated camera pose relative to tool0 -->
@@ -122,6 +122,6 @@
       <!-- Origin is tool0 -> camera (meters, radians).
           RPY is extrinsic X-Y-Z (roll, pitch, yaw) as in URDF. -->
-      <origin xyz="-0.004171269533157492 0.3005070159435434 -0.05050934664329281"
-               rpy="1.4706191997841613 -0.011294149359347028 -3.108643277714379"/>
+      <origin xyz="-0.0026397426633640534 0.2998884350074318 -0.046887903327791254"
+               rpy="1.4738212164540254 -0.004557843376089332 -3.1083688441677833"/>
     </joint>
     <!-- Fixed frame for calibrated Extruder tcp pose relative to tool0 -->
@@ -132,5 +132,5 @@
       <!-- Origin is tool0 -> extruder(meters, radians).
           RPY is extrinsic X-Y-Z (roll, pitch, yaw) as in URDF. -->
-      <origin xyz="-0.00391 0.47471 0.08024"
+      <origin xyz="-0.00448 0.4728 0.08175"
               rpy="1.5641113421 0.0 0.0"/>
     </joint>

Commit message: print segments update

File: src/custom_workcell/ur20_workcell/urdf/workcell_macro.xacro (robot description, xacro)
@@ -112,6 +112,6 @@
       <!-- Origin is tool0 -> camera (meters, radians).
           RPY is extrinsic X-Y-Z (roll, pitch, yaw) as in URDF. -->
-      <origin xyz="-0.034063681747165384 0.2956667467761771 -0.04632604563225764"
-               rpy="1.5797083152416658 -0.0024684364752196597 -3.109366333302816"/>
+      <origin xyz="-0.03237220097014208 0.2975795037710782 -0.049440132645135075"
+               rpy="1.5737478510469156 -0.00037951050418594257 -3.129989760064829"/>
     </joint>
     <!-- Fixed frame for calibrated camera pose relative to tool0 -->
@@ -122,6 +122,6 @@
       <!-- Origin is tool0 -> camera (meters, radians).
           RPY is extrinsic X-Y-Z (roll, pitch, yaw) as in URDF. -->
-      <origin xyz="-0.0026397426633640534 0.2998884350074318 -0.046887903327791254"
-               rpy="1.4738212164540254 -0.004557843376089332 -3.1083688441677833"/>
+      <origin xyz="0.0001260989423124842 0.299380885120948 -0.048070702286223926"
+               rpy="1.4679434434594152 -0.004381501036235358 -3.1293804627485198"/>
     </joint>
     <!-- Fixed frame for calibrated Extruder tcp pose relative to tool0 -->
@@ -132,5 +132,5 @@
       <!-- Origin is tool0 -> extruder(meters, radians).
           RPY is extrinsic X-Y-Z (roll, pitch, yaw) as in URDF. -->
-      <origin xyz="-0.00448 0.4728 0.08175"
+      <origin xyz="-0.00551 0.47304 0.0822"
               rpy="1.5641113421 0.0 0.0"/>
     </joint>

Commit message: calibration tcp and cameras

File: src/custom_workcell/ur20_workcell/urdf/workcell_macro.xacro (robot description, xacro)
@@ -112,6 +112,6 @@
       <!-- Origin is tool0 -> camera (meters, radians).
           RPY is extrinsic X-Y-Z (roll, pitch, yaw) as in URDF. -->
-      <origin xyz="-0.03237220097014208 0.2975795037710782 -0.049440132645135075"
-               rpy="1.5737478510469156 -0.00037951050418594257 -3.129989760064829"/>
+      <origin xyz="-0.027418302205691688 0.2981950632445194 -0.04833072930568825"
+               rpy="1.5671126183823887 0.001219177107494085 3.122301119125984"/>
     </joint>
     <!-- Fixed frame for calibrated camera pose relative to tool0 -->
@@ -122,6 +122,6 @@
       <!-- Origin is tool0 -> camera (meters, radians).
           RPY is extrinsic X-Y-Z (roll, pitch, yaw) as in URDF. -->
-      <origin xyz="0.0001260989423124842 0.299380885120948 -0.048070702286223926"
-               rpy="1.4679434434594152 -0.004381501036235358 -3.1293804627485198"/>
+      <origin xyz="0.004908790432333231 0.30002747459759455 -0.04965832990331366"
+               rpy="1.4588805414160293 -0.0016304370242608002 3.1246897752124143"/>
     </joint>
     <!-- Fixed frame for calibrated Extruder tcp pose relative to tool0 -->
@@ -132,5 +132,5 @@
       <!-- Origin is tool0 -> extruder(meters, radians).
           RPY is extrinsic X-Y-Z (roll, pitch, yaw) as in URDF. -->
-      <origin xyz="-0.00551 0.47304 0.0822"
+      <origin xyz="0.00368 0.47435 0.09141"
               rpy="1.5641113421 0.0 0.0"/>
     </joint>

Commit message: calibrated camera

File: src/custom_workcell/ur20_workcell/urdf/workcell_macro.xacro (robot description, xacro)
@@ -112,6 +112,6 @@
       <!-- Origin is tool0 -> camera (meters, radians).
           RPY is extrinsic X-Y-Z (roll, pitch, yaw) as in URDF. -->
-      <origin xyz="-0.027418302205691688 0.2981950632445194 -0.04833072930568825"
-               rpy="1.5671126183823887 0.001219177107494085 3.122301119125984"/>
+      <origin xyz="-0.025515490322922284 0.2992429004009513 -0.04776767499425601"
+               rpy="1.5745245745971501 -0.0009563747551801782 3.1213800188359433"/>
     </joint>
     <!-- Fixed frame for calibrated camera pose relative to tool0 -->
@@ -122,6 +122,6 @@
       <!-- Origin is tool0 -> camera (meters, radians).
           RPY is extrinsic X-Y-Z (roll, pitch, yaw) as in URDF. -->
-      <origin xyz="0.004908790432333231 0.30002747459759455 -0.04965832990331366"
-               rpy="1.4588805414160293 -0.0016304370242608002 3.1246897752124143"/>
+      <origin xyz="0.005752294662071668 0.30167909897409373 -0.04898595730658378"
+               rpy="1.4671078814465028 -0.004127058062504796 3.122566426149098"/>
     </joint>
     <!-- Fixed frame for calibrated Extruder tcp pose relative to tool0 -->
@@ -132,5 +132,5 @@
       <!-- Origin is tool0 -> extruder(meters, radians).
           RPY is extrinsic X-Y-Z (roll, pitch, yaw) as in URDF. -->
-      <origin xyz="0.00368 0.47435 0.09141"
+      <origin xyz="0.0037 0.47356 0.09103"
               rpy="1.5641113421 0.0 0.0"/>
     </joint>

Commit message: tcp calib

File: src/custom_workcell/ur20_workcell/urdf/workcell_macro.xacro (robot description, xacro)
@@ -132,5 +132,5 @@
       <!-- Origin is tool0 -> extruder(meters, radians).
           RPY is extrinsic X-Y-Z (roll, pitch, yaw) as in URDF. -->
-      <origin xyz="0.0037 0.47356 0.09103"
+      <origin xyz="0.00508 0.47425 0.09026"
               rpy="1.5641113421 0.0 0.0"/>
     </joint>
